File: V1.0/KiCAD/V1.0/V1.0.kicad_sch (KiCad schematic)
At the start: 55 parts, among them IC1 TL494CN, IC2 XC7S6-1FTGB196I, J1 Conn_01x02_Socket, J2 Conn_01x02_Socket, Q1 BD139, Q2 IRFP250PBF, Q3 NMOS, Q4 NMOS, Q5 NMOS, Q6 NMOS

Commit message: More Parts added to the Schematic
Parts:
- added C26, C30, C31: 4u7, symbol Device:C
- added C27: 3n5, symbol Device:C
- added C28: 620p, symbol Device:C
- added C29, C33, C35: 10u, symbol Device:C
- added C32: 14n, symbol Device:C
- added C34: 100n, symbol Device:C
- added IC3, IC4, IC5: LM3671MF-1.8_NOPB, SOT95P280X145-5N, symbol LM3671MF-1.8:LM3671MF-1.8_NOPB
- added IC6: FT2232H-56Q-REEL, QFN50P800X800X100-57N-D, symbol FT2232H:FT2232H-56Q-REEL
- added IC7: MT25QL256ABA8ESF-0AAT, SOIC127P1032X265-16N, symbol MT25QL256:MT25QL256ABA8ESF-0AAT
- added J3: 12401832E402A, 12401832E402A, symbol 12401832E402A:12401832E402A
- added L4, L5, L6: 2u2, symbol Device:L
- added R16, R17: 5k1, symbol Device:R_US
- added R18, R22, R23: 1k, symbol Device:R_US
- added R19: 5k6, symbol Device:R_US
- added R20: 10k, symbol Device:R_US
- added R21: 26k, symbol Device:R_US
- added R24: 10R, symbol Device:R_US
- added R25, R26: 22R, symbol Device:R_US
- added U1: KC2520Z, Oscillator:Oscillator_SMD_Kyocera_KC2520Z-4Pin_2.5x2.0mm, symbol Oscillator:KC2520Z
Connections:
- net +12V: now also C26.2, C27.1, C29.2, C30.2, C31.2, C33.2, C34.1, C35.2, IC3.2 (GND), IC4.2 (GND), IC5.2 (GND), IC7.10 (VSS), J3.A1 (GND_1), J3.A12 (GND_2), J3.B1 (GND_3), J3.B12 (GND_4), R16.2, R17.2, R18.1, R20.1, R22.1, U1.2 (GND)
- net +1V0: now also C35.1, L6.2, R23.2
- net +1V8: now also C32.2, C33.1, L5.2, R21.2
- net +3V3: now also C28.2, C29.1, C34.2, IC7.2 (VCC), L4.2, R19.2, U1.1 (INH), U1.4 (VCC)
- net at IC2.H4 (IO_L13P_T2_MRCC_34): now also R24.2
- net MOSFET4: now reaches IC2.L3 (IO_L22P_T3_34)
- net MOSFET1: now reaches IC2.M1 (IO_L18P_T2_34)
- net MOSFET2: now reaches IC2.M3 (IO_L19P_T3_34)
- net MOSFET3: now reaches IC2.M5 (IO_L23P_T3_34)
- new net: IC3.5 (SW), L4.1
- new net: J3.A5 (CC1), R17.1
- new net: J3.B5 (CC2), R16.1
- new net: IC5.4 (FB), R22.2, R23.1
- new net: IC5.5 (SW), L6.1
- new net: C27.2, C28.1, IC3.4 (FB), R18.2, R19.1
- new net: R24.1, U1.3 (CLK)
- new net: IC7.16 (C), R25.1
- new net: IC7.3 (RESET#), R26.2
- new net: C32.1, IC4.4 (FB), R20.2, R21.1
- new net: IC4.5 (SW), L5.1
- new net QSPI DATA0: IC7.15 (DQ0)
- new net QSPI DATA1: IC7.8 (DQ1)
- new net QSPI DATA2: IC7.9 (W#/DQ2)
- new net QSPI DATA3: IC7.1 (DQ3/HOLD#)
- new net QSPI NSS: IC7.7 (S#)
- new net QSPI RESET: R26.1
- new net QSPI SCLK: R25.2
- new net VBUS1: C26.1, IC3.1 (VIN), IC3.3 (EN), J3.A4 (VBUS_1)
- new net VBUS2: C30.1, IC4.1 (VIN), IC4.3 (EN), J3.A9 (VBUS_2)
- new net VBUS3: C31.1, IC5.1 (VIN), IC5.3 (EN), J3.B4 (VBUS_3)
- no-connect marks 7 -> 14

Commit message: Schematic is Finished
Parts:
- added C36: 0u1, symbol Device:C
- added R27: 10k, symbol Device:R_US
- added R28: 12k±1%, symbol Device:R_US
Connections:
- net +12V: now also IC6.10 (TEST), IC6.21 (GND_1), IC6.41 (GND_2), IC6.45 (GND_3), C36.2, R28.1
- net +3V3: now also R27.1
- net QSPI DATA0: now also IC2.B11 (IO_L1P_T0_D00_MOSI_14)
- net QSPI DATA1: now also IC2.B12 (IO_L1N_T0_D01_DIN_14)
- net QSPI DATA2: now also IC2.D10 (IO_L2P_T0_D02_14)
- net QSPI DATA3: now also IC2.C10 (IO_L2N_T0_D03_14)
- net QSPI SCLK: now also IC2.A8 (CCLK_0)
- net VBUS1: no longer C26.1, IC3.1 (VIN), J3.A4 (VBUS_1)
- net VBUS2: no longer C30.1, IC4.1 (VIN), J3.A9 (VBUS_2)
- net VBUS3: no longer C31.1, IC5.1 (VIN), J3.B4 (VBUS_3)
- net USB_P: now reaches J3.A6 (D+_1)
- net USB_P: now also IC6.8 (DP), J3.B6 (D+_2)
- net USB_N: now reaches J3.A7 (D-_1)
- net USB_N: now also IC6.7 (DM), J3.B7 (D-_2)
- net +5V: now reaches J3.B9 (VBUS_4)
- net +5V: now also C26.1, C30.1, C31.1, IC3.1 (VIN), IC4.1 (VIN), IC5.1 (VIN), IC6.43 (VREGOUT), IC6.44 (VREGIN), J3.A4 (VBUS_1), J3.A9 (VBUS_2), J3.B4 (VBUS_3)
- net TCK: now reaches IC2.A7 (TCK_0)
- net TCK: now also IC6.12 (ADBUS0)
- net 12MCLK: now reaches IC2.H4 (IO_L13P_T2_MRCC_34), R24.2
- net 12MCLK: now also IC6.3 (OSCI)
- net TMS: now reaches IC2.M6 (TMS_0)
- net TMS: now also IC6.15 (ADBUS3)
- net TDO: now reaches IC2.P6 (TDO_0)
- net TDO: now also IC6.14 (ADBUS2)
- net TDI: now reaches IC2.P7 (TDI_0)
- net TDI: now also IC6.13 (ADBUS1)
- net RESET: now reaches IC6.11 (RESET#)
- net RESET: now also C36.1, R27.2
- net +3.3V: now reaches IC6.16 (VCCIO_1)
- net +3.3V: now also IC6.2 (VCORE_1), IC6.31 (VCORE_2), IC6.36 (VCCIO_2), IC6.5 (VPHY), IC6.9 (VPLL)
- net at IC6.6 (REF): now also R28.2
- no-connect marks 14 -> 15
Other:
- moved on the sheet: C34, IC7, R16, R17, R24, R25, R26, U1

Commit message: Update To Schematic
Parts:
- removed J1: Conn_01x02_Socket, symbol Connector:Conn_01x02_Socket
- removed R26: 22R, symbol Device:R_US
- added C37, C38: 0u22, symbol Device:C
- added C39, C40: 4u7, symbol Device:C
- added C41: 100n, symbol Device:C
- added IC8: MAX662AESA+T, SOIC127P600X175-8N, symbol MAX662AESA:MAX662AESA+T
- added R29: 4k7, symbol Device:R_US
- added R30: 1k, symbol Device:R_US
- added R31, R32, R33: 12k, symbol Device:R_US
- C25: value C -> 2uF
- L2, L3: value L -> 900mH
- R15: value R_US -> 900
Connections:
- net VBUS1 is gone; now on net +5V: IC3.3 (EN)
- net VBUS2 is gone; now on net +5V: IC4.3 (EN)
- net VBUS3 is gone; now on net +5V: IC5.3 (EN)
- net +12V: now also IC2.E6 (GND_21), IC2.M8 (M1_0), IC2.M9 (M2_0), C39.2, C40.1, C40.2, C41.2, IC8.6 (VOUT), IC8.7 (GND), IC8.8 (SHDN)
- net +3V3: now also IC2.G2 (VCCO_34_1), C41.1, R29.2, R30.2, R31.2, R32.2, R33.2
- net +5V: now also C39.1, IC8.5 (VCC)
- net MOSFET1: now also Q3.2 (G)
- net MOSFET2: now also Q4.2 (G)
- net MOSFET3: now also Q5.2 (G)
- net MOSFET4: now also Q6.2 (G)
- net QSPI DATA2: now also R32.1
- net QSPI DATA3: now also R31.1
- net QSPI NSS: now also IC2.C11 (IO_L6P_T0_FCS_B_14), R33.1
- net at IC2.M7 (M0_0): now also R30.1
- net at IC2.P8 (INIT_B_0): now also R29.1
- net +120V renamed 120V
- net MOS1: no longer names the net of IC2.A3 (IO_L2N_T0_34)
- net MOS1: no longer Q3.2 (G)
- net MOS2: no longer names the net of IC2.B1 (IO_L5N_T0_34)
- net MOS2: no longer Q4.2 (G)
- net MOS3: no longer names the net of IC2.C3 (IO_L1N_T0_34)
- net MOS3: no longer Q5.2 (G)
- net MOS4: no longer names the net of IC2.A5 (IO_L4N_T0_34)
- net MOS4: no longer Q6.2 (G)
- new net: C38.1, IC8.3 (C2-)
- new net: C38.2, IC8.4 (C2+)
- new net: C37.1, IC8.1 (C1-)
- new net: C37.2, IC8.2 (C1+)
- no-connect marks 15 -> 160
Other:
- note added: "12MHz Clock and QSPI Flash"
- note added: "Boost Converter and H-Bridge"
- note added: "FPGA Banks with Decoupling Capacitors"
- note added: "USB-C and Power Regulators"
- note added: "USB-C to JTAG"
- moved on the sheet: C1, C10, C11, C12, C13, C14, C15, C16, C17, C18, C19, C2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
