File: V1.0/KiCAD/V1.0/V1.0.kicad_sch (KiCad schematic)
At the start: 98 parts, among them IC1 TL494CN, IC2 XC7S6-1FTGB196I, IC3 LM3671MF-1.8_NOPB, IC4 LM3671MF-1.8_NOPB, IC5 LM3671MF-1.8_NOPB, IC6 FT2232H-56Q-REEL, IC7 MT25QL256ABA8ESF-0AAT, IC8 MAX662AESA+T, J2 Conn_01x02_Socket, J3 12401832E402A, Q1 BD139, Q2 IRFP250PBF, Q3 NMOS, Q4 NMOS, Q5 NMOS, Q6 NMOS, U1 KC2520Z

Commit message: PCB Design is almost finished.
Parts:
- removed C37, C38: 0u22, symbol Device:C
- removed C39, C40: 4u7, symbol Device:C
- removed IC8: MAX662AESA+T, SOIC127P600X175-8N, symbol MAX662AESA:MAX662AESA+T
- removed J3: 12401832E402A, 12401832E402A, symbol 12401832E402A:12401832E402A
- removed R16, R17: 5k1, symbol Device:R_US
- removed RV1: 100k, symbol Device:R_Potentiometer_US
- added C42: 47u, KGM21AR51A476MU:CAPC2012X145N, symbol Device:C
- added D2: MBRS130T3G, MBRS130T3G:DIOM5436X247N, symbol MBRS130T3G:MBRS130T3G
- added IC9: LT1111CS8-5#PBF, LT1111CS8:SOIC127P599X175-8N, symbol LT1111CS8:LT1111CS8-5#PBF
- added J1: 12401948E412A, 12401948E412A:AMPHENOL_12401948E412A, symbol 12401948E412A:12401948E412A
- added J3: Conn_01x02_Socket, Connector_Phoenix_MSTB:PhoenixContact_MSTBA_2,5_2-G_1x02_P5.00mm_Horizontal, symbol Connector:Conn_01x02_Socket
- added L7: 68uH, 744772680:WE-TI_809589, symbol Device:L
- added R26: 1k, 3503G2B1K0FTDF:RESC3016X58N, symbol Device:R_US
- added R34, R35: 5k1, ERJ-UP6D5101V:ERJUP6, symbol Device:R_US
- added VR1: PCW1D-C24-KAB104L, PCW1D-C24-KAB104L:PCW1DC24KAB104L, symbol PCW1D-C24-KAB104L:PCW1D-C24-KAB104L
- C1, C34, C36, C41: footprint (none) -> KAM15AR71H104KM:CAPC1608X90N
- C10, C11, C12, C13, C19, C20, C21, C24: footprint (none) -> KAF31ER71H474KL:CAPC3216X152N
- C14, C15, C18, C23, C26, C30, C31, C9: footprint (none) -> GCJ188C70J475KE02:CAPC1608X100N
- C16, C17, C8: footprint (none) -> KGM21AR51A476MU:CAPC2012X145N
- C2: footprint (none) -> CAPC2012X140N:CAPC2012X140N
- C22: footprint (none) -> MAL2142231101E3:CAPPRD350W60D850H1300
- C25: value 2uF -> 1uF; footprint (none) -> KAM03CT70J105KH:CAPC0603X39N
- C27, C5: footprint (none) -> C0805C362G4HACTU:C0805
- C28: footprint (none) -> C0603C621F5GACTU:CAPC1608X87N
- C29, C33, C35: footprint (none) -> KAF32LR71H106KL:CAPC3225X178N
- C3: footprint (none) -> KAF21BR72D102KT:CAPC2012X94N
- C32: footprint (none) -> C2220C143KFGLCAUTO:CAPC5750X550N
- C4, C6: footprint (none) -> C0402C101KCGACA:CAPC1005X55N
- C7: footprint (none) -> KAM15AR72A103KM:CAPC1608X90N
- D1: footprint (none) -> 15ETH06:TO508P465X1031X1932-2P
- IC1: footprint DIP794W53P254L1930H508Q16N -> TL494CN:DIP794W53P254L1930H508Q16N
- IC2: footprint BGA196C100P14X14_1500X1500X155 -> XC7S6-1FTGB196I:BGA196C100P14X14_1500X1500X155
- IC3, IC4, IC5: footprint SOT95P280X145-5N -> LM3671MF-1:SOT95P280X145-5N
- IC6: footprint QFN50P800X800X100-57N-D -> FT2232H:QFN50P800X800X100-57N-D
- IC7: footprint SOIC127P1032X265-16N -> MT25QL256ABA8ES:SOIC127P1032X265-16N
- J2: footprint (none) -> Connector_Phoenix_MSTB:PhoenixContact_MSTBA_2,5_2-G_1x02_P5.00mm_Horizontal
- L1: footprint (none) -> SRR5228A-221M:SRR5228A
- L2, L3: value 900mH -> 100mH; footprint (none) -> 19R107C:CAPPRD600W90D1200H2100
- L4, L5, L6: footprint (none) -> RCH875NP-2R2M:RCH875NP2R2M
- Q2: footprint TO546P531X1558X2511-3P -> IRF640PBF:TO254P465X1024X2050-3P
- Q3, Q4, Q5, Q6: footprint (none) -> IRF640PBF:TO254P465X1024X2050-3P
- R1, R3: footprint (none) -> MCS04020D4702BE:RESC1005X37N
- R10, R30, R9: footprint (none) -> ERA-8VEB4700V:ERA8KEB1004V
- R11, R20, R27: footprint (none) -> MCS0402MD1002B:RESC1005X37N
- R12: footprint (none) -> CRCW04022K20DH:RESC1005X40N
- R13: footprint (none) -> ERJ-UP6D2702V:ERJUP6
- R14: footprint (none) -> ERJ-1GJF6802C:ERJ1GJJ2R4C
- R15: footprint (none) -> RT1206CRE07900R:RESC3116X65N
- R18, R22, R23, R6: footprint (none) -> 3503G2B1K0FTDF:RESC3016X58N
- R19: footprint (none) -> ERA-2ARBS62X:ERA2AED122X
- R2: footprint (none) -> ERJ-UP6D6802V:ERJUP6
- R21: footprint (none) -> ERA-2ARB2612X:ERA2AED122X
- R24: footprint (none) -> TNPW120610R0BEE:RESC3216X65N
- R25: footprint (none) -> CRCW120622R0JNE:RESC3116X65N
- R28, R31, R32, R33, R7: footprint (none) -> ERA-8VRB1202V:ERA8KEB1004V
- R29: footprint (none) -> ERA-3ARB472V:ERA3AEB101V
- R4, R5: footprint (none) -> ERA-8VRB2202V:ERA8KEB1004V
- R8: footprint (none) -> WSLP5931L1000FEA:RESC15077X100N
Connections:
- net +12V: now also C42.2, D2.2 (A), IC9.2 (VIN), IC9.3 (SW1), IC9.5 (GND), J1.A12_B1 (GND), J1.A1_B12 (GND), J1.S1 (SHELL_GND), J1.S2 (SHELL_GND), J1.S3 (SHELL_GND), J1.S4 (SHELL_GND), J3.1 (Pin_1), J3.2 (Pin_2), R26.1, R34.2, R35.2
- net +5V: now also C42.1, IC9.8 (SENSE), J1.A4_B9 (VBUS), J1.A9_B4 (VBUS), L7.1
- net USB_N: now also J1.A7 (D1-), J1.B7 (D2-)
- net USB_P: now also J1.A6 (D1+), J1.B6 (D2+)
- net at R11.2: now also VR1.1 (CCW)
- net at IC1.16 (2IN+): now also VR1.2 (WIPER)
- net at R12.1: now also VR1.3 (CW)
- new net: D2.1 (K), IC9.4 (SW2), L7.2
- new net: IC9.1 (ILIM), R26.2
- new net: J1.A5 (CC1), R34.1
- new net: J1.B5 (CC2), R35.1
- no-connect marks 160 -> 154
Other:
- moved on the sheet: R12

Commit message: Finished the PCB Design!
Connections:
- net +5V: no longer J1.A4_B9 (VBUS), J1.A9_B4 (VBUS)
- new net: J1.A4_B9 (VBUS), J1.A9_B4 (VBUS)
- no-connect marks 154 -> 155
Changed lines of the file:
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@@
 	)
 	(no_connect
+		(at 104.14 68.58)
+	)
+	(no_connect
 		(at 330.2 69.85)
 	)
@@
 	(wire
 		(pts
-			(xy 107.95 68.58) (xy 107.95 67.31)
-		)
-		(stroke
-			(width 0)
-			(type default)
-		)
-	)
-	(wire
-		(pts
 			(xy 179.07 173.99) (xy 180.34 173.99)
 		)
@@
 	(wire
 		(pts
-			(xy 104.14 68.58) (xy 107.95 68.58)
-		)
-		(stroke
-			(width 0)
-			(type default)
-		)
-	)
-	(wire
-		(pts
 			(xy 72.39 438.15) (xy 72.39 440.69)
 		)
@@
 					(unit 1)
 				)
-			)
-		)
-	)
-	(symbol
-		(lib_id "power:+5V")
-		(at 107.95 67.31 0)
-		(unit 1)
-		(exclude_from_sim no)
-		(in_bom yes)
-		(on_board yes)
-		(dnp no)
-		(fields_autoplaced yes)
-		(property "Reference" "#PWR097"
-			(at 107.95 71.12 0)
-			(effects
-				(font
-					(size 1.27 1.27)
-				)
-				(hide yes)
-			)
-		)
-		(property "Value" "+5V"
-			(at 107.95 62.23 0)
-			(effects
-				(font
-					(size 1.27 1.27)
-				)
-			)
-		)
-		(property "Footprint" ""
-			(at 107.95 67.31 0)
-			(effects
-				(font
-					(size 1.27 1.27)
-				)
-				(hide yes)
-			)
-		)
-		(property "Datasheet" ""
-			(at 107.95 67.31 0)
-			(effects
-				(font
-					(size 1.27 1.27)
-				)
-				(hide yes)
-			)
-		)
-		(property "Description" "Power symbol creates a global label with name \"+5V\""
-			(at 107.95 67.31 0)
-			(effects
-				(font
-					(size 1.27 1.27)
-				)
-				(hide yes)
-			)
-		)
-		(pin "1"
-		)
-		(instances
-			(project "V1.0"
-				(path "/53b2a5be-9ef4-49a8-af7b-42525ecf0c9a"
-					(reference "#PWR097")
-					(unit 1)
-				)
