File: V1.0/KiCAD/V1.0/V1.0.kicad_pcb (KiCad board)
At the start: 4 copper layers, 9.8 x 4.5 mm, 99 parts, among them IC1 TL494CN, IC2 XC7S6-1FTGB196I, IC3 LM3671MF-1.8_NOPB, IC4 LM3671MF-1.8_NOPB, IC5 LM3671MF-1.8_NOPB, IC6 FT2232H-56Q-REEL, IC7 MT25QL256ABA8ESF-0AAT, IC9 LT1111CS8-5#PBF, J1 12401948E412A, J2 Conn_01x02_Socket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

Commit message: Added Images
Parts:
- moved C31 16.7 mm to (121.2, 130.7)
- moved C12 16.7 mm to (130.1, 128.8)
- moved R23 16.7 mm to (112.0, 135.6)
- moved R4 16.7 mm to (146.0, 65.3)
- moved VR1 16.7 mm to (171.0, 41.3)
- moved C1 16.7 mm to (141.2, 91.0)
- moved C11 16.7 mm to (130.1, 132.0)
- moved C13 16.7 mm to (130.1, 125.7)
- moved C14 16.7 mm to (130.4, 122.7)
- moved C15 16.7 mm to (130.4, 120.3)
- moved C16 16.7 mm to (130.2, 118.2)
- moved C17 16.7 mm to (135.2, 123.1)
- moved C18 16.7 mm to (135.1, 121.1)
- moved C19 16.7 mm to (134.7, 118.6)
- moved C2 16.7 mm to (135.4, 65.2)
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Routing:
- added copper zone on B.Cu, net +12V
Other:
- board size 9.8 x 4.5 mm -> 105 x 132.5 mm

Commit message: Finished the PCB Design!
Connections:
- IC6 pad 16: +3.3V -> +3V3
- IC6 pad 31: +3.3V -> +3V3
- IC6 pad 36: +3.3V -> +3V3
- IC6 pad 9: +3.3V -> +3V3
- J1 pad A4_B9: +5V -> unconnected-(J1-VBUS-PadA4_B9)_0
- J1 pad A9_B4: +5V -> unconnected-(J1-VBUS-PadA4_B9)
Routing:
- net +1V0: track 34.2 -> 194.4 mm, vias 0 -> 2
- net +1V8: track 101.8 -> 260.3 mm, vias 3 -> 5
- net +5V: track 60.2 -> 182.7 mm, vias 6 -> 5
- net +3V3: track 188.8 -> 298.7 mm, vias 7 -> 11
- net /120V: track 40.6 -> 126.3 mm, vias 0 -> 2
- net +12V: track 404.8 -> 481.3 mm, vias 14 -> 27
- net /MOSFET4: track 2.22 -> 54.7 mm
- net /MOSFET3: track 2.22 -> 51.5 mm, vias 1 -> 2
- net Net-(J2-Pin_2): track 22.9 -> 55.0 mm
- net /USB_P: track 2.94 -> 34.2 mm
- net /USB_N: track 2.98 -> 33.8 mm
- net /TMS: track 0.00 -> 21.8 mm
- net Net-(IC1-REF): track 31.3 -> 50.7 mm, vias 0 -> 2
- net Net-(Q1-C): track 7.45 -> 26.5 mm, vias 0 -> 2
- net /MOSFET2: track 36.7 -> 54.2 mm
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Other:
- board text removed: "12V"
